Commit message: Add files via upload
This is the update till date for the bipedal bot after adding controllers and imu

File: final_assem2/urdf/final_assem2.urdf (robot description, URDF)
Before this commit: robot final_assem2, 11 links, 10 joints
Links:
- removed link left_upper2_leg
- removed link left_upper_leg
- removed link right_upper2_leg
- removed link right_upper_leg
- added link imu_link, mass 0.0001
- link base_link: mass 0.159950800266572 -> 0.0001
- link left_lower_leg: mass 0.0110711596178799 -> 0.0001
- link left_wheel: mass 0.0821704328344352 -> 2.5
- link left_white_link: mass 0.0136561818789523 -> 0.0001
- link right_lower_leg: mass 0.0110711602724557 -> 0.0001
- link right_wheel: mass 0.0821706301013002 -> 2.5
- link right_white_link: mass 0.0136561811410979 -> 0.0001
Joints:
- removed joint left_hip_joint 
- removed joint left_upper_bottom_joint
- removed joint right_hip_joint
- removed joint right_upper_bottom_joint
- added joint imu_joint: type fixed, parent base_link, child imu_link, origin xyz=0 0 0.05 rpy=0 0 0
- joint left_wheel_joint: axis -1 0 0 -> 1 0 0; limit effort=10 velocity=5 -> effort=1000 velocity=20
- joint left_white_bottom_joint: limit lower=-1.5708 upper=1.5708 effort=10 velocity=1 -> lower=-1.5708 upper=1.5708 effort=1000 velocity=1
- joint left_white_top_joint: limit lower=-1.5708 upper=1.5708 effort=10 velocity=1 -> lower=-1.5708 upper=1.5708 effort=1000 velocity=1
- joint right_wheel_joint: axis -1 0 0 -> 1 0 0; limit effort=10 velocity=5 -> effort=1000 velocity=20
- joint right_white_bottom_joint: limit lower=-1.5708 upper=1.5708 effort=10 velocity=1 -> lower=-1.5708 upper=1.5708 effort=1000 velocity=1
- joint right_white_top_joint: limit lower=-1.5708 upper=1.5708 effort=10 velocity=1 -> lower=-1.5708 upper=1.5708 effort=1000 velocity=1
